Commit message: 対面環境(dqn)学習データの追加

File: urdf_dumps/robot_1.urdf (robot description, URDF)
Before this commit: robot turtlebot4, 23 links, 22 joints
Links:
- removed link imu_link
Joints:
- removed joint imu_joint

File: urdf_dumps/robot_10.urdf (robot description, URDF)
Before this commit: robot turtlebot4, 23 links, 22 joints
Links:
- removed link imu_link
Joints:
- removed joint imu_joint

File: urdf_dumps/robot_11.urdf (robot description, URDF)
Before this commit: robot turtlebot4, 22 links, 21 joints
Links:
- added link imu_link, mass 0.01
Joints:
- added joint imu_joint: type fixed, parent base_link, child imu_link, origin xyz=0.050613 0.043673 0.0844

File: urdf_dumps/robot_12.urdf (robot description, URDF)
Before this commit: robot turtlebot4, 22 links, 21 joints
Links:
- added link imu_link, mass 0.01
Joints:
- added joint imu_joint: type fixed, parent base_link, child imu_link, origin xyz=0.050613 0.043673 0.0844

File: urdf_dumps/robot_13.urdf (robot description, URDF)
Before this commit: robot turtlebot4, 22 links, 21 joints
Links:
- added link imu_link, mass 0.01
Joints:
- added joint imu_joint: type fixed, parent base_link, child imu_link, origin xyz=0.050613 0.043673 0.0844

File: urdf_dumps/robot_14.urdf (robot description, URDF)
Before this commit: robot turtlebot4, 22 links, 21 joints
Links:
- added link imu_link, mass 0.01
Joints:
- added joint imu_joint: type fixed, parent base_link, child imu_link, origin xyz=0.050613 0.043673 0.0844

File: urdf_dumps/robot_15.urdf (robot description, URDF)
Before this commit: robot turtlebot4, 22 links, 21 joints
Links:
- added link imu_link, mass 0.01
Joints:
- added joint imu_joint: type fixed, parent base_link, child imu_link, origin xyz=0.050613 0.043673 0.0844

File: urdf_dumps/robot_16.urdf (robot description, URDF)
Before this commit: robot turtlebot4, 22 links, 21 joints
Links:
- added link imu_link, mass 0.01
Joints:
- added joint imu_joint: type fixed, parent base_link, child imu_link, origin xyz=0.050613 0.043673 0.0844

File: urdf_dumps/robot_17.urdf (robot description, URDF)
Before this commit: robot turtlebot4, 22 links, 21 joints
Links:
- added link imu_link, mass 0.01
Joints:
- added joint imu_joint: type fixed, parent base_link, child imu_link, origin xyz=0.050613 0.043673 0.0844

File: urdf_dumps/robot_18.urdf (robot description, URDF)
Before this commit: robot turtlebot4, 22 links, 21 joints
Links:
- added link imu_link, mass 0.01
Joints:
- added joint imu_joint: type fixed, parent base_link, child imu_link, origin xyz=0.050613 0.043673 0.0844

File: urdf_dumps/robot_19.urdf (robot description, URDF)
Before this commit: robot turtlebot4, 22 links, 21 joints
Links:
- added link imu_link, mass 0.01
Joints:
- added joint imu_joint: type fixed, parent base_link, child imu_link, origin xyz=0.050613 0.043673 0.0844

File: urdf_dumps/robot_2.urdf (robot description, URDF)
Before this commit: robot turtlebot4, 23 links, 22 joints
Links:
- removed link imu_link
Joints:
- removed joint imu_joint

File: urdf_dumps/robot_20.urdf (robot description, URDF)
Before this commit: robot turtlebot4, 22 links, 21 joints
Links:
- added link imu_link, mass 0.01
Joints:
- added joint imu_joint: type fixed, parent base_link, child imu_link, origin xyz=0.050613 0.043673 0.0844

File: urdf_dumps/robot_3.urdf (robot description, URDF)
Before this commit: robot turtlebot4, 23 links, 22 joints
Links:
- removed link imu_link
Joints:
- removed joint imu_joint

File: urdf_dumps/robot_4.urdf (robot description, URDF)
Before this commit: robot turtlebot4, 23 links, 22 joints
Links:
- removed link imu_link
Joints:
- removed joint imu_joint

File: urdf_dumps/robot_5.urdf (robot description, URDF)
Before this commit: robot turtlebot4, 23 links, 22 joints
Links:
- removed link imu_link
Joints:
- removed joint imu_joint

File: urdf_dumps/robot_6.urdf (robot description, URDF)
Before this commit: robot turtlebot4, 23 links, 22 joints
Links:
- removed link imu_link
Joints:
- removed joint imu_joint

File: urdf_dumps/robot_7.urdf (robot description, URDF)
Before this commit: robot turtlebot4, 23 links, 22 joints
Links:
- removed link imu_link
Joints:
- removed joint imu_joint

File: urdf_dumps/robot_8.urdf (robot description, URDF)
Before this commit: robot turtlebot4, 23 links, 22 joints
Links:
- removed link imu_link
Joints:
- removed joint imu_joint

File: urdf_dumps/robot_9.urdf (robot description, URDF)
Before this commit: robot turtlebot4, 23 links, 22 joints
Links:
- removed link imu_link
Joints:
- removed joint imu_joint
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