Commit message: train/c/dqn学習結果の追加

File: src/tb4_launcher/urdf/icreate/caster.urdf.xacro (robot description, xacro)
@@ -11,11 +11,10 @@
   </joint>
   <link name="${name}_link">
-    <visual>
+    <!-- <visual>
       <geometry>
         <sphere radius="${radius}"/>
       </geometry>
-      <!-- Give black color to caster in Rviz -->
       <xacro:insert_block name="material_black"/>
-    </visual>
+    </visual> -->
     <collision>
       <geometry>
@@ -34,5 +33,5 @@
   </gazebo>
   <gazebo reference="${name}_link">
-    <material>Gazebo/DarkGrey</material>
+    <xacro:material_darkgray/>
     <mu1>0.1</mu1>
     <mu2>0.1</mu2>

File: src/tb4_launcher/urdf/icreate/common_properties.urdf.xacro (robot description, xacro)
@@ -82,5 +82,5 @@
   <!-- Material colors -->
   <xacro:property name="material_black">
-    <material name="black">
+    <material name="icreate_black">
       <color rgba="0.1 0.1 0.1 1"/>
     </material>

File: src/tb4_launcher/urdf/icreate/create3.urdf.xacro (robot description, xacro)
@@ -129,42 +129,14 @@
         <update_rate>30</update_rate>
       </plugin>
-        <gazebo>
-          <plugin name="ground_truth" filename="libgazebo_ros_p3d.so">
-            <frameName>map</frameName>
-            <bodyName>base_footprint</bodyName>
-            <topicName>$(arg namespace)/tracker</topicName>
-            <updateRate>10.0</updateRate>
-          </plugin>
-        </gazebo>
-      <!-- <plugin
-        filename="gz-sim-odometry-publisher-system"
-        name="gz::sim::systems::OdometryPublisher">
-        <dimensions>3</dimensions>
-        <odom_frame>map</odom_frame>
-        <robot_base_frame>base_footprint</robot_base_frame>
-        <publish_tf>true</publish_tf>
-        <update_rate>50</update_rate>
-      </plugin> -->
-      <!-- <plugin name="ground_truth_p3d" filename="libgazebo_ros_p3d.so">
-        <ros>
-          <remapping>/tf:=$(arg namespace)/tf</remapping>
-          <remapping>/tf_static:=$(arg namespace)/tf_static</remapping>
-        </ros>
-        <tf_topic>$(arg namespace)/tf</tf_topic>
-        <body_name>${frame_prefix}base_footprint</body_name>
-        <frame_name>${frame_prefix}odom</frame_name>
-        <update_rate>50.0</update_rate>
-        <xyz_offset>0 0 0</xyz_offset>
-        <rpy_offset>0 0 0</rpy_offset>
-        <gaussian_noise>0.0</gaussian_noise>
-      </plugin> -->
-      <!-- <plugin
-        filename="gz-sim-odometry-publisher-system"
-        name="gz::sim::systems::OdometryPublisher">
-        <dimensions>3</dimensions>
-        <tf_topic>$(arg namespace)/tf</tf_topic>
-        <odom_frame>${frame_prefix}odom</odom_frame>
-        <robot_base_frame>${frame_prefix}base_footprint</robot_base_frame>
-        <publish_tf>true</publish_tf>
+      <!-- <plugin filename="gz-sim-pose-publisher-system" name="gz::sim::systems::PosePublisher">
+        <publish_link_pose>false</publish_link_pose>
+        <publish_sensor_pose>false</publish_sensor_pose>
+        <publish_collision_pose>false</publish_collision_pose>
+        <publish_visual_pose>false</publish_visual_pose>
+        <publish_nested_model_pose>false</publish_nested_model_pose>
+        <publish_model_pose>true</publish_model_pose>
+        <use_pose_vector_msg>true</use_pose_vector_msg>
+        <static_publisher>true</static_publisher>
+        <static_update_frequency>1</static_update_frequency>
       </plugin> -->
   </gazebo>

File: src/tb4_launcher/urdf/icreate/wheel.urdf.xacro (robot description, xacro)
@@ -41,5 +41,5 @@
     <minDepth>0.0001</minDepth>
     <maxVel>1.0</maxVel>
-    <material>Gazebo/DarkGrey</material>
+    <xacro:material_darkgray/>
   </gazebo>
 </xacro:macro>

File: urdf_dumps/robot_1.urdf (robot description, URDF)
Before this commit: robot turtlebot4, 22 links, 21 joints
Links:
- link front_caster_link: geometry collision sphere radius=0.01

File: urdf_dumps/robot_2.urdf (robot description, URDF)
Before this commit: robot turtlebot4, 22 links, 21 joints
Links:
- link front_caster_link: geometry collision sphere radius=0.01

File: urdf_dumps/robot_3.urdf (robot description, URDF)
Before this commit: robot turtlebot4, 22 links, 21 joints
Links:
- link front_caster_link: geometry collision sphere radius=0.01

File: urdf_dumps/robot_4.urdf (robot description, URDF)
Before this commit: robot turtlebot4, 22 links, 21 joints
Links:
- link front_caster_link: geometry collision sphere radius=0.01

File: urdf_dumps/robot_5.urdf (robot description, URDF)
Before this commit: robot turtlebot4, 22 links, 21 joints
Links:
- link front_caster_link: geometry collision sphere radius=0.01

File: urdf_dumps/robot_6.urdf (robot description, URDF)
Before this commit: robot turtlebot4, 22 links, 21 joints
Links:
- link front_caster_link: geometry collision sphere radius=0.01

File: urdf_dumps/robot_7.urdf (robot description, URDF)
Before this commit: robot turtlebot4, 22 links, 21 joints
Links:
- link front_caster_link: geometry collision sphere radius=0.01

File: urdf_dumps/robot_8.urdf (robot description, URDF)
Before this commit: robot turtlebot4, 22 links, 21 joints
Links:
- link front_caster_link: geometry collision sphere radius=0.01
